File: board/board.kicad_pcb (KiCad board)
At the start: 2 copper layers, 21 x 13 mm, 1 part

Commit message: initial
Parts:
- added J1: 020_1000BASE-T_with_CT, on_edge:on_edge_2x10_host, F.Cu at (174.0, 56.0)
- added J2: 003_power, on_edge:on_edge_2x05_device, F.Cu at (129.0, 56.0)
- added J3: 008_USB, on_edge:on_edge_2x05_device, F.Cu at (129.0, 88.0)
- added J4: 001_I2C, on_edge:on_edge_2x05_host, F.Cu at (174.0, 136.0)
- added J5: 008_USB, on_edge:on_edge_2x05_host, F.Cu at (174.0, 104.0)
- added J6: 002_SPI, on_edge:on_edge_2x05_host, F.Cu at (174.0, 120.0)
- added J7: 010_UART, on_edge:on_edge_2x05_host, F.Cu at (174.0, 88.0)
- added R1: 0R, Resistor_SMD:R_0603_1608Metric, F.Cu at (165.0, 154.0)
- added R2: 0R, Resistor_SMD:R_0603_1608Metric, F.Cu at (172.5, 152.0)
- added R3: 560R, Resistor_SMD:R_0603_1608Metric, F.Cu at (172.5, 156.0)
- added R4: d.n.p, Resistor_SMD:R_0603_1608Metric, F.Cu at (175.0, 156.0)
- added U1: VAR-SOM, b107:TE_1473149-4, F.Cu at (141.0, 87.5)
- moved LOGO1 37.4 mm to (132.1, 66.2)
Routing:
- net GND: track 0.00 -> 51.3 mm
- net /var-som/ETH_A_MDI_B-: track 0.00 -> 41.4 mm
- net /var-som/ETH_A_MDI_B+: track 0.00 -> 40.8 mm
- net /var-som/ETH_A_MDI_A-: track 0.00 -> 40.1 mm
- net /var-som/ETH_A_MDI_A+: track 0.00 -> 39.3 mm
- net /var-som/USB_A_D-: track 0.00 -> 32.8 mm, vias 0 -> 2
- net /UART5_RX: track 0.00 -> 32.2 mm, vias 0 -> 2
- net /var-som/USB_A_D+: track 0.00 -> 31.4 mm, vias 0 -> 2
- net /var-som/ETH_A_MDI_D-: track 0.00 -> 31.0 mm
- net /UART5_TX: track 0.00 -> 30.7 mm, vias 0 -> 2
- net /var-som/ETH_A_MDI_D+: track 0.00 -> 30.4 mm
- net /var-som/ETH_A_MDI_C-: track 0.00 -> 30.1 mm
- net /var-som/ETH_A_MDI_C+: track 0.00 -> 29.5 mm
- net /var-som/USB_B_D+: track 0.00 -> 16.2 mm, vias 0 -> 2
- net /var-som/USB_B_D-: track 0.00 -> 16.1 mm, vias 0 -> 2
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Other:
- board size 21 x 13 mm -> 45 x 94 mm
